File: PCB/ReflowControllerREV1/ReflowControllerREV1.kicad_pcb (KiCad board)
At the start: 2 copper layers, 73.7 x 61 mm, 39 parts, among them IC1 MOC3020, J1 Fan_CONN, J2 Thermocouple_CONN, J3 AC_CONN, J4 HEATER_CONN, J5 CONN_AC_to_12v400mA, J6 ENCODER_CONN, J7 TFT_CONN, Q1 IRF540N, Q2 BT137, U1 H11AA1-X007T, U2 MAX6675ISA+

Commit message: firmware finished
Routing:
- net GND: track 6.78 -> 15.1 mm
Changed lines of the file:
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@@
     (thickness 1.6)
     (drawings 48)
-    (tracks 301)
+    (tracks 305)
     (zones 0)
     (modules 39)
@@
       (rotate (xyz 0 0 0))
     )
+    (model ${KIPRJMOD}/3DModels/Terminal5mmx2.stp
+      (offset (xyz -3 -3 0))
+      (scale (xyz 1 1 1))
+      (rotate (xyz -90 0 90))
+    )
   )
   (module TerminalBlock:TerminalBlock_bornier-2_P5.08mm (layer F.Cu)
@@
       (net 41 AC1_IN))
     (model ${KISYS3DMOD}/TerminalBlock.3dshapes/TerminalBlock_bornier-2_P5.08mm.wrl
-      (offset (xyz 2.539999961853027 0 0))
-      (scale (xyz 1 1 1))
-      (rotate (xyz 0 0 0))
+      (offset (xyz 2.54 0 0))
+      (scale (xyz 1 1 1))
+      (rotate (xyz 10 0 0))
+    )
+    (model ${KIPRJMOD}/3DModels/Terminal5mmx2.stp
+      (offset (xyz -3 -3.5 0))
+      (scale (xyz 1 1 1))
+      (rotate (xyz -90 0 90))
     )
   )
@@
       (rotate (xyz 0 0 0))
     )
+    (model ${KIPRJMOD}/3DModels/SOIC-8_3,9x4,9.STEP
+      (at (xyz 0 0 0))
+      (scale (xyz 1 1 1))
+      (rotate (xyz 0 0 90))
+    )
   )
   (module Package_DIP:DIP-6_W7.62mm_LongPads (layer F.Cu)
@@
       (scale (xyz 1 1 1))
       (rotate (xyz 0 0 0))
+    )
+    (model ${KIPRJMOD}/3DModels/Arduino_nano.STEP
+      (offset (xyz 0 0 1.5))
+      (scale (xyz 1 1 1))
+      (rotate (xyz -90 0 90))
     )
   )
@@
   (segment (start 200.913692 114.350492) (end 199.8472 113.284) (width 0.25) (layer F.Cu) (net 7))
   (segment (start 201.061628 114.350492) (end 200.913692 114.350492) (width 0.25) (layer F.Cu) (net 7))
+  (segment (start 199.484999 74.516999) (end 195.993001 74.516999) (width 0.25) (layer F.Cu) (net 7))
+  (segment (start 200.66 75.692) (end 199.484999 74.516999) (width 0.25) (layer F.Cu) (net 7))
+  (segment (start 195.993001 74.516999) (end 195.58 74.93) (width 0.25) (layer F.Cu) (net 7))
+  (segment (start 195.58 74.93) (end 195.58 77.47) (width 0.25) (layer F.Cu) (net 7))
   (segment (start 198.354001 107.422001) (end 207.264 116.332) (width 0.5) (layer F.Cu) (net 8))
   (segment (start 190.773999 106.772001) (end 191.423999 107.422001) (width 0.5) (layer F.Cu) (net 8))

Commit message: final pcb
Parts:
- removed C3: 10n, Capacitor_SMD:C_0805_2012Metric_Pad1.15x1.40mm_HandSolder
- removed G***: LOGO, CTB_Logo:KicadCTBLogo
- removed R11, R13, R15, R17, R9: 20k, Resistor_SMD:R_0805_2012Metric_Pad1.15x1.40mm_HandSolder
- removed R6: 180, Resistor_SMD:R_0805_2012Metric_Pad1.15x1.40mm_HandSolder
- removed REF**: OSHW-Logo_11.4x12mm_SilkScreen, Symbol:OSHW-Logo_11.4x12mm_SilkScreen
- R10, R12, R14, R16, R8: value 10k -> 1k
- moved R5 2.83 mm to (238.5, 99.1), turned to 180 degrees
- moved R1 0.51 mm to (214.9, 94.5)
- turned R2 to 180 degrees
Connections:
- C4 pad 2: TC2 -> GND
- J2 pad 2: TC2 -> GND
- Q1 pad 2: GND -> Net-(D1-Pad2)
- Q1 pad 3: Net-(D1-Pad2) -> GND
- R2 pad 1: Net-(Q1-Pad1) -> GND
- R2 pad 2: GND -> Net-(Q1-Pad1)
- R5 pad 1: Net-(C3-Pad1) -> AC1_OUT
- R5 pad 2: AC1_IN -> Net-(IC1-Pad6)
- U2 pad 2: TC2 -> GND
Routing:
- net GND: track 15.1 -> 104.0 mm, vias 5 -> 1
- net TC2: track 15.2 -> 0.00 mm
- net Net-(C3-Pad1): track 7.25 -> 0.00 mm
- net Net-(IC1-Pad6): track 3.47 -> 8.98 mm
- net CS_: track 17.7 -> 12.6 mm
- net AC1_OUT: track 18.8 -> 21.0 mm
- net AC1_IN: track 55.9 -> 53.9 mm
