File: PCB/ReflowControllerREV1/ReflowControllerREV1.sch (KiCad schematic (older format))
At the start: 37 parts, among them IC1 MOC3020, J1 Fan_CONN, J2 Thermocouple_CONN, J3 AC_CONN, J4 HEATER_CONN, J5 CONN_AC_to_12v400mA, J6 ENCODER_CONN, J7 TFT_CONN, Q1 IRF540N, Q2 BT137, U1 H11AA1-X007T, U2 MAX6675ISA+

Commit message: firmware finished
Changed lines of the file:
@@
 EESchema Schematic File Version 4
-LIBS:ReflowControllerREV1-cache
 EELAYER 30 0
 EELAYER END
@@
 Connection ~ 8200 3350
 NoConn ~ 4550 3750
+Entry Wire Line
+	200  4550 300  4650
+Entry Wire Line
+	200  4550 300  4650
 $EndSCHEMATC

Commit message: schematic updated
Parts:
- removed C3: 10n, Capacitor_SMD:C_0805_2012Metric_Pad1.15x1.40mm_HandSolder, symbol Device:C
- removed R11, R13, R15, R17, R9: 20k, Resistor_SMD:R_0805_2012Metric_Pad1.15x1.40mm_HandSolder, symbol Device:R
- removed R5: 2.4k, Resistor_SMD:R_0805_2012Metric_Pad1.15x1.40mm_HandSolder, symbol Device:R
- removed R6: 180, Resistor_SMD:R_0805_2012Metric_Pad1.15x1.40mm_HandSolder, symbol Device:R
- added R?: 2.4k, Resistor_SMD:R_0805_2012Metric_Pad1.15x1.40mm_HandSolder, symbol Device:R
- A1: symbol MCU_Module:Arduino_Nano_v3.x -> ReflowControllerREV1-rescue:Arduino_Nano_v3.x-MCU_Module
- R10, R12, R14, R16, R8: value 10k -> 1k
Connections:
- net TC2 is gone; now on net GND: C4.2, J2.2, U2.2 (T-)
- net AC1_OUT: now also R?.1
- net GND: now also Q1.3 (S), R2.1; no longer Q1.2 (D), R2.2
- net at BZ1.1 (-): now also A1.15 (D12); no longer A1.26 (A7)
- net at IC1.6 (A2): now also R?.2
- net at D1.2 (A), J1.2 (-): now also Q1.2 (D); no longer Q1.3 (S)
- net at Q1.1 (G), R1.1: now also R2.2; no longer R2.1
Other:
- moved on the sheet: BZ1, D1, J1, R2

Commit message: final pcb
Parts:
- gave numbers to parts that had none: 1
Connections:
- net at BZ1.1 (-): now also A1.26 (A7); no longer A1.15 (D12)
Other:
- note added: "5v to 3.3v"
- moved on the sheet: BZ1, R12
Changed lines of the file:
@@
 $EndComp
 Wire Notes Line
-	5750 4750 8350 4750
-Wire Notes Line
-	8350 4750 8350 2650
-Wire Notes Line
-	8350 2650 5750 2650
+	8700 4750 8700 2650
 Wire Notes Line
 	5750 2650 5750 4750
@@
 L Device:R R12
 U 1 1 5DDFD1A4
-P 10000 1950
-F 0 "R12" H 10070 1996 50  0000 L CNN
-F 1 "1k" H 10070 1905 50  0000 L CNN
-F 2 "Resistor_SMD:R_0805_2012Metric_Pad1.15x1.40mm_HandSolder" V 9930 1950 50  0001 C CNN
-F 3 "~" H 10000 1950 50  0001 C CNN
-	1    10000 1950
-	1    0    0    -1
-$EndComp
-Text GLabel 10150 2150 2    50   Input ~ 0
+P 9100 5800
+F 0 "R12" H 9170 5846 50  0000 L CNN
+F 1 "1k" H 9170 5755 50  0000 L CNN
+F 2 "Resistor_SMD:R_0805_2012Metric_Pad1.15x1.40mm_HandSolder" V 9030 5800 50  0001 C CNN
+F 3 "~" H 9100 5800 50  0001 C CNN
+	1    9100 5800
+	1    0    0    -1
+$EndComp
+Text GLabel 9250 6000 2    50   Input ~ 0
 SCK
 Wire Wire Line
-	10150 2150 10000 2150
-Wire Wire Line
-	10000 2150 10000 2100
-Text GLabel 10000 1750 1    50   Input ~ 0
+	9250 6000 9100 6000
+Wire Wire Line
+	9100 6000 9100 5950
+Text GLabel 9100 5600 1    50   Input ~ 0
 SCK_5
 Wire Wire Line
-	10000 1800 10000 1750
+	9100 5650 9100 5600
 Text GLabel 1850 4750 0    50   Input ~ 0
 SCK_5
@@
 Connection ~ 8200 3350
 NoConn ~ 4550 3750
-Entry Wire Line
-	200  4550 300  4650
-Entry Wire Line
-	200  4550 300  4650
-$Comp
-L power:GND #PWR?
+$Comp
+L power:GND #PWR0101
 U 1 1 5EFBEAB6
 P 6200 4050
-F 0 "#PWR?" H 6200 3800 50  0001 C CNN
+F 0 "#PWR0101" H 6200 3800 50  0001 C CNN
 F 1 "GND" H 6205 3877 50  0000 C CNN
 F 2 "" H 6200 4050 50  0001 C CNN
@@
 L Device:Buzzer BZ1
 U 1 1 5D1349AA
-P 1650 5150
-F 0 "BZ1" H 1802 5179 50  0000 L CNN
-F 1 "Buzzer" H 1802 5088 50  0000 L CNN
-F 2 "Connector_PinHeader_2.54mm:PinHeader_1x02_P2.54mm_Vertical" V 1625 5250 50  0001 C CNN
-F 3 "~" V 1625 5250 50  0001 C CNN
-	1    1650 5150
+P 3300 4850
+F 0 "BZ1" H 3452 4879 50  0000 L CNN
+F 1 "Buzzer" H 3452 4788 50  0000 L CNN
+F 2 "Connector_PinHeader_2.54mm:PinHeader_1x02_P2.54mm_Vertical" V 3275 4950 50  0001 C CNN
+F 3 "~" V 3275 4950 50  0001 C CNN
+	1    3300 4850
 	1    0    0    -1
 $EndComp
@@
 L power:GND #PWR09
 U 1 1 5D1653E8
-P 1500 5300
-F 0 "#PWR09" H 1500 5050 50  0001 C CNN
-F 1 "GND" H 1505 5127 50  0000 C CNN
-F 2 "" H 1500 5300 50  0001 C CNN
-F 3 "" H 1500 5300 50  0001 C CNN
-	1    1500 5300
-	1    0    0    -1
-$EndComp
-Wire Wire Line
-	1550 5250 1500 5250
-Wire Wire Line
-	1500 5250 1500 5300
-Wire Wire Line
-	1550 5050 1350 5050
-Wire Wire Line
-	1350 5050 1350 4650
-Wire Wire Line
-	1350 4650 2000 4650
-$Comp
-L Device:R R?
+P 3150 5000
+F 0 "#PWR09" H 3150 4750 50  0001 C CNN
+F 1 "GND" H 3155 4827 50  0000 C CNN
+F 2 "" H 3150 5000 50  0001 C CNN
+F 3 "" H 3150 5000 50  0001 C CNN
+	1    3150 5000
+	1    0    0    -1
+$EndComp
+Wire Wire Line
+	3200 4950 3150 4950
+Wire Wire Line
+	3150 4950 3150 5000
+Wire Wire Line
+	3200 4750 3000 4750
+$Comp
+L Device:R R5
 U 1 1 5EFD62C2
 P 6000 1700
-F 0 "R?" V 5793 1700 50  0000 C CNN
+F 0 "R5" V 5793 1700 50  0000 C CNN
 F 1 "2.4k" V 5884 1700 50  0000 C CNN
 F 2 "Resistor_SMD:R_0805_2012Metric_Pad1.15x1.40mm_HandSolder" V 5930 1700 50  0001 C CNN
@@
 	2400 6750 2400 6650
 $Comp
-L power:GND #PWR?
+L power:GND #PWR0102
 U 1 1 5F00C1FF
 P 2850 7050
-F 0 "#PWR?" H 2850 6800 50  0001 C CNN
+F 0 "#PWR0102" H 2850 6800 50  0001 C CNN
 F 1 "GND" H 2700 6950 50  0000 C CNN
 F 2 "" H 2850 7050 50  0001 C CNN
@@
 Wire Wire Line
 	2850 6300 2850 6200
+Wire Notes Line
+	8700 2650 5750 2650
+Wire Notes Line
+	5750 4750 8700 4750
+Wire Notes Line
+	8900 2650 11100 2650
+Wire Notes Line
+	11100 2650 11100 6400
+Wire Notes Line
+	11100 6400 8500 6400
+Wire Notes Line
+	8500 6400 8500 4900
+Wire Notes Line
+	8500 4900 8900 4900
+Wire Notes Line
+	8900 4900 8900 2650
+Text Notes 8900 2650 0    50   ~ 0
+5v to 3.3v
 $EndSCHEMATC
